File: Pico Version/PiDG_Pico.kicad_sch (KiCad schematic)
At the start: 48 parts, among them J1 Conn_02x05_Odd_Even, J10 Trig, J11 Laser Enable, J12 Pixel Reset, J13 Debug, J2 Conn_02x05_Odd_Even, J3 Conn_02x05_Odd_Even, J4 Conn_02x05_Odd_Even, J5 Conn_02x05_Odd_Even, J6 Conn_02x05_Odd_Even, J7 Laser 1, J8 Laser 2, U1 74LVC1G04, U10 74LVC1G08, U11 Raspberry Pi Pico, U12 74LVC1G08, U13 UCC27524, U2 SN74LVC04AD, U3 74LVC1G04, U4 SN74LVC04AD, U5 74LVC1G04, U6 SN74LVC04AD, U7 74LVC1G08, U8 74LVC1G08, U9 NCP718xSN180

Commit message: Update project for Pico 2 W RP2350
Parts:
- U11: value Raspberry Pi Pico -> Raspberry Pi Pico 2 W
Changed lines of the file:
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@@
 			)
 		)
-		(property "Value" "Raspberry Pi Pico"
+		(property "Value" "Raspberry Pi Pico 2 W"
 			(at 103 283 0)
 			(effects
@@
 			)
 		)
-		(property "Datasheet" "https://datasheets.raspberrypi.com/pico/pico-datasheet.pdf"
+		(property "Datasheet" "https://datasheets.raspberrypi.com/picow/pico-2-w-datasheet.pdf"
 			(at 100 280 0)
 			(effects
@@
 			)
 		)
-		(property "Description" "RP2040 module -- replaces the Teensy 4.1 (see HARDWARE_DESIGN.md)"
+		(property "Description" "RP2350 + CYW43439 (wireless unused) module -- replaces the Teensy 4.1 (see HARDWARE_DESIGN.md)"
 			(at 100 280 0)
 			(effects

Commit message: AI been working at it
Parts:
- U11: footprint (none) -> RPi_Pico:RPi_Pico2W_SMD_TH
Changed lines of the file:
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@@
 			)
 		)
-		(property "Footprint" ""
+		(property "Footprint" "RPi_Pico:RPi_Pico2W_SMD_TH"
 			(at 100 280 0)
 			(effects

Commit message: Mor AI workings
Connections:
- net +3V3: now also U11.36 (3V3_OUT); no longer U11.25 (GND)
- net +5V: now also U11.39 (VSYS), U11.40 (VBUS), U13.1 (ENA), U13.6 (VDD), U13.8 (ENB); no longer U11.21 (GP16), U13.4 (INB), U13.5 (OUTB), U13.7 (OUTA)
- net CH1_DRIVE_RAW: now also U13.7 (OUTA); no longer U13.6 (VDD)
- net CH1_GATED: now also U13.2 (INA); no longer U13.3 (GND)
- net CH2_DRIVE_RAW: now also U13.5 (OUTB); no longer U13.8 (ENB)
- net CH2_GATED: now also U13.4 (INB); no longer U13.1 (ENA)
- net GND: now also J13.2 (Pin_2), J7.2 (Ext), J8.2 (Ext), U11.25 (GND), U11.42 (GND), U13.3 (GND); no longer U13.2 (INA)
- net at U11.41 (SWCLK): now also J13.1 (Pin_1)
- net at U11.43 (SWDIO): now also J13.3 (Pin_3)
- no-connect marks 80 -> 81
