File: Pico Version 4Layer/PiDG_Pico.kicad_pcb (KiCad board)
At the start: 4 copper layers, 126 x 126 mm, 70 parts, among them J1 Conn_02x05_Odd_Even, J10 Trig, J11 Laser Enable, J12 Pixel Reset, J14 Pico Socket A, J15 Pico Socket B, J16 Laser En/PWM Trig/GND, J17 USB-C PD in, J2 Conn_02x05_Odd_Even, J3 Conn_02x05_Odd_Even, J4 Conn_02x05_Odd_Even, J5 Conn_02x05_Odd_Even, J6 Conn_02x05_Odd_Even, J7 Laser 1, J8 Laser 2, U1 74LVC1G04, U10 74AHCT1G08, U12 74LVC1G17, U13 UCC27524, U14 CH224K, U15 AP63205WU, U16 LM66100, U17 LP2951D, U2 SN74LVC04AD, U3 74LVC1G04, U4 SN74LVC04AD, U5 74LVC1G04, U6 SN74LVC04AD, U7 74AHCT1G08, U8 74AHCT1G08, U9 NCP718xSN180

Commit message: Update KiCad hardware and schematic design
Parts:
- 1MHz Clock: renamed from TP3
Other:
- board text added: "LASER 1 (50Ohm)"
- board text added: "LASER 2 (50 Ohm)"
- board text removed: "LASER 1"
- board text removed: "LASER 2"
Changed lines of the file:
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@@
 		(descr "Through hole angled pin header, 1x02, 2.54mm pitch, 6mm pin length, single row")
 		(tags "Through hole angled pin header THT 1x02 2.54mm single row")
-		(property "Reference" "TP3"
-			(at -2.907 0 90)
+		(property "Reference" "1MHz Clock"
+			(at 0.063171 -5.762076 0)
 			(layer "F.SilkS")
 			(effects
@@
 		)
 	)
+	(gr_text "GND"
+		(at 159.74 34.53 0)
+		(layer "F.SilkS")
+		(effects
+			(font
+				(size 1 1)
+				(thickness 0.15)
+			)
+			(justify left bottom)
+		)
+	)
 	(gr_text "ENABLE"
 		(at 245.24 55.03 0)
@@
 		)
 	)
-	(gr_text "PIXEL RESET"
-		(at 234.24 127.53 0)
+	(gr_text "LASER 2 (50 Ohm)"
+		(at 233.24 107.03 0)
 		(layer "F.SilkS")
 		(effects
@@
 		)
 	)
-	(gr_text "LASER 2"
-		(at 235.74 107.53 0)
+	(gr_text "LASER 1 (50Ohm)"
+		(at 233.74 87.03 0)
 		(layer "F.SilkS")
 		(effects
@@
 		)
 	)
-	(gr_text "LASER 1"
-		(at 236.74 87.03 0)
+	(gr_text "PIXEL RESET"
+		(at 234.24 127.53 0)
 		(layer "F.SilkS")
 		(effects
