File: Pico Version 4Layer/PiDG_Pico.kicad_sch (KiCad schematic)
At the start: 67 parts, among them J1 Conn_02x05_Odd_Even, J10 Trig, J11 Laser Enable, J12 Pixel Reset, J14 Pico Socket A, J15 Pico Socket B, J16 Laser En/PWM Trig/GND, J17 USB-C PD in, J2 Conn_02x05_Odd_Even, J3 Conn_02x05_Odd_Even, J4 Conn_02x05_Odd_Even, J5 Conn_02x05_Odd_Even, J6 Conn_02x05_Odd_Even, J7 Laser 1, J8 Laser 2, U1 74LVC1G04, U10 74AHCT1G08, U11 Raspberry Pi Pico 2 W, U12 74LVC1G17, U13 UCC27524, U14 CH224K, U15 AP63205WU, U16 LM66100, U17 LP2951D, U2 SN74LVC04AD, U3 74LVC1G04, U4 SN74LVC04AD, U5 74LVC1G04, U6 SN74LVC04AD, U7 74AHCT1G08, U8 74AHCT1G08, U9 NCP718xSN180

Commit message: Update KiCad hardware and schematic design
Other:
- company: DLR Insitute of Propulsion Technology -> (none)
- title: IDS EVS Event-camera Synchronizer -> IDS EVS Event-camera Synchronizer (Pico 2)
