File: Pico Version 4Layer/PiDG_Pico.kicad_sch (KiCad schematic)
At the start: 81 parts, among them J1 Conn_02x05_Odd_Even, J10 Trig, J11 Laser Enable, J12 Pixel Reset, J14 Pico Socket A, J15 Pico Socket B, J16 Laser En/PWM Trig/GND, J17 USB-C PD in, J18 Laser 1 mode, J19 Laser 2 mode, J2 Conn_02x05_Odd_Even, J3 Conn_02x05_Odd_Even, J4 Conn_02x05_Odd_Even, J5 Conn_02x05_Odd_Even, J6 Conn_02x05_Odd_Even, J7 Laser 1, J8 Laser 2, U1 74LVC1G04, U10 74AHCT1G08, U11 Raspberry Pi Pico 2 W, U12 74LVC1G17, U13 UCC27524, U14 CH224A, U15 AP63205WU, U16 LM66100, U17 LT3065EDD, U18 TPS3700DDC, U2 SN74LVC04AD, U3 74LVC1G00, U4 SN74LVC04AD, U5 74LVC1G04, U6 SN74LVC04AD, U7 74AHCT1G08, U8 74AHCT1G08, U9 NCP718xSN180

Commit message: JLC cost-down and laser amplitude margin for the Pico board
Availability and cost (JLC data of 2026-10-05):
- U9: NCP718BSN180T1G (C892792), in stock; NCP718ASN180T1G has none.
  Same datasheet, pinout and +/-2 % 1.8 V output. Pre-order: 162 pcs.
- R25/R26: Yageo AC2512FK-7W47RL (C7209419), higher stock.
- U18 divider R21/R22/R23 -> 150k / 1.2k / 4.7k, all JLC basic parts
  (removes two extended lines).

Laser amplitude margin:
- U13 (UCC27524, SOIC-8 D package) has ROH 5 typ / 8.5 max ohm with no
  minimum (SLUSFA9), not the 2.5-7.5 ohm used before. With 101k the 50 ohm
  high corner reached 5.19 V (0.3 % below the 5.2 V limit).
- R12 101k -> 100k 0.1 % (C122537): +12V is 11.8 V (11.54-12.05 V), and the
  50 ohm output is 4.54-5.14 V (0.8 % / 1.2 % margin). Hi-Z mode 4.55-5.08 V.
- U18 retuned for the new rail: UV 10.6 V rising (release <= 10.89 V,
  0.65 V below the rail band), OV 13.3 V (12.88-13.67 V, 0.82 V above it).
- The DSD package (ROH 2.5-7.5 ohm) was rejected: 25 ns max minimum pulse
  width and 4 ns channel matching break the 20 ns WIDTH and 1-2 ns matching.

Docs, BOMs, CPL, README and schematic notes updated. ERC/DRC: no new
findings against the previous commit; gerbers unchanged.

Co-Authored-By: Claude Opus 5.5 <noreply@anthropic.com>
Parts:
- R12: value 101k -> 100k
- R21: value 1M -> 150k
- R22: value 6.04k -> 1.2k
- R23: value 31.6k -> 4.7k
Other:
- note added: "Output mode, one shunt per channel (J18 = Laser 1, J19 = Laser 2): 1-2 50 ohm: series 47R bypassed. 4.54-5.14 V into a 50 ohm load (PicoLas LDP-V); ~12 V open circuit. 2-3 Hi-Z: 68R + 47R in series, 82R shunt -> 4.55-5.08 V open circuit from a 47-50 ohm source (back-terminated, no overshoot on long cables); 2.3-2.6 V into 50 ohm: an LDP-V will not trigger. No shunt: ~12 V open circuit, ~3.5 V int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"
- note added: "U17: 11.8 V laser rail, 400 mA limit (R20). U18 (sheet bottom left) holds U13 disabled (LASER_PWR_OK low) unless +12V is inside 10.6-13.3 V (TPS3700 window)."
- note added: "USB-C PD input. U14 requests 15 V. U15 buck + U16 ideal diode feed the +5V plane (Pico VSYS). U17 makes the 11.8 V +12V rail for U13; U18 gates U13's enables (see the note by U17). Pico VBUS is NOT on +5V: USB reaches VSYS only through the Pico's own Schottky."
- note removed: "Output mode, one shunt per channel (J18 = Laser 1, J19 = Laser 2): 1-2 50 ohm: series 47R bypassed. 4.61-5.08 V into a 50 ohm load (PicoLas LDP-V); ~12 V open circuit. 2-3 Hi-Z: 68R + 47R in series, 82R shunt -> 4.62-5.06 V open circuit from a 48-50 ohm source (back-terminated, no overshoot on long cables); 2.3-2.6 V into 50 ohm: an LDP-V will not trigger. No shunt: ~12 V open circuit, ~3.5 V int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"
- note removed: "U17: 11.9 V laser rail, 400 mA limit (R20). U18 (sheet bottom left) holds U13 disabled (LASER_PWR_OK low) unless +12V is inside 11.0-13.1 V (TPS3700 window)."
- note removed: "USB-C PD input. U14 requests 15 V. U15 buck + U16 ideal diode feed the +5V plane (Pico VSYS). U17 makes the 11.9 V +12V rail for U13; U18 gates U13's enables (see the note by U17). Pico VBUS is NOT on +5V: USB reaches VSYS only through the Pico's own Schottky."
Changed lines of the file:
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@@
 		(comment 2 "Chris Willert")
 	)
-	(text "USB-C PD input. U14 requests 15 V. U15 buck + U16 ideal diode feed the +5V plane (Pico VSYS).\nU17 makes the 11.9 V +12V rail for U13; U18 gates U13's enables (see the note by U17).\nPico VBUS is NOT on +5V: USB reaches VSYS only through the Pico's own Schottky."
+	(text "USB-C PD input. U14 requests 15 V. U15 buck + U16 ideal diode feed the +5V plane (Pico VSYS).\nU17 makes the 11.8 V +12V rail for U13; U18 gates U13's enables (see the note by U17).\nPico VBUS is NOT on +5V: USB reaches VSYS only through the Pico's own Schottky."
 		(exclude_from_sim no)
 		(at 308.356 232.918 0)
@@
 		)
 	)
-	(text "Output mode, one shunt per channel (J18 = Laser 1, J19 = Laser 2):\n  1-2  50 ohm: series 47R bypassed. 4.61-5.08 V into a 50 ohm load (PicoLas LDP-V); ~12 V open circuit.\n  2-3  Hi-Z: 68R + 47R in series, 82R shunt -> 4.62-5.06 V open circuit from a 48-50 ohm source\n       (back-terminated, no overshoot on long cables); 2.3-2.6 V into 50 ohm: an LDP-V will not trigger.\n  No shunt: ~12 V open circuit, ~3.5 V into 50 ohm. Ship with both shunts on 1-2."
+	(text "Output mode, one shunt per channel (J18 = Laser 1, J19 = Laser 2):\n  1-2  50 ohm: series 47R bypassed. 4.54-5.14 V into a 50 ohm load (PicoLas LDP-V); ~12 V open circuit.\n  2-3  Hi-Z: 68R + 47R in series, 82R shunt -> 4.55-5.08 V open circuit from a 47-50 ohm source\n       (back-terminated, no overshoot on long cables); 2.3-2.6 V into 50 ohm: an LDP-V will not trigger.\n  No shunt: ~12 V open circuit, ~3.5 V into 50 ohm. Ship with both shunts on 1-2."
 		(exclude_from_sim no)
 		(at 122 217.17 0)
@@
 		)
 	)
-	(text "U17: 11.9 V laser rail, 400 mA limit (R20).\nU18 (sheet bottom left) holds U13 disabled\n(LASER_PWR_OK low) unless +12V is inside\n11.0-13.1 V (TPS3700 window)."
+	(text "U17: 11.8 V laser rail, 400 mA limit (R20).\nU18 (sheet bottom left) holds U13 disabled\n(LASER_PWR_OK low) unless +12V is inside\n10.6-13.3 V (TPS3700 window)."
 		(exclude_from_sim no)
 		(at 240.03 252.73 0)
@@
 			)
 		)
-		(property "Description" "Series resistor, 2 W 2512. 50 ohm mode (J19 on 1-2): 11.9 V x 50/(50+68+ROH) = 4.61-5.08 V into the 50 ohm LDP-V trigger input"
+		(property "Description" "Series resistor, 2 W 2512. 50 ohm mode (J19 on 1-2): 11.8 V x 50/(50+68+ROH) = 4.54-5.14 V into the 50 ohm LDP-V trigger input (ROH 0-8.5 ohm)"
 			(at 400.05 39.37 0)
 			(hide yes)
@@
 			)
 		)
-		(property "Description" "12 V laser rail: 45 V / 500 mA LDO. VOUT = 0.6 V x (1 + R12/R13) = 11.9 V. R20 sets a 400 mA current limit."
+		(property "Description" "12 V laser rail: 45 V / 500 mA LDO. VOUT = 0.6 V x (1 + R12/R13) = 11.8 V. R20 sets a 400 mA current limit."
 			(at 266.7 220.98 0)
 			(hide yes)
@@
 			)
 		)
-		(property "Description" "Series resistor, 2 W 2512. 50 ohm mode (J18 on 1-2): 11.9 V x 50/(50+68+ROH) = 4.61-5.08 V into the 50 ohm LDP-V trigger input"
+		(property "Description" "Series resistor, 2 W 2512. 50 ohm mode (J18 on 1-2): 11.8 V x 50/(50+68+ROH) = 4.54-5.14 V into the 50 ohm LDP-V trigger input (ROH 0-8.5 ohm)"
 			(at 400.05 44.45 0)
 			(hide yes)
@@
 			)
 		)
-		(property "Value" "101k"
+		(property "Value" "100k"
 			(at 286.004 217.17 0)
 			(show_name no)
@@
 			)
 		)
-		(property "Description" "LT3065 feedback top, 0.1 % thin film: 11.906 V = 0.6 V x (1 + 101k/5.36k)"
+		(property "Description" "LT3065 feedback top, 0.1 % thin film: 11.794 V = 0.6 V x (1 + 100k/5.36k)"
 			(at 284.48 215.9 0)
 			(hide yes)
@@
 			)
 		)
-		(property "Description" "Laser power-good: OUTA low if +12V < 11.0 V (UV), OUTB low if +12V > 13.1 V (OV). Drives U13 ENA/ENB."
+		(property "Description" "Laser power-good: OUTA low if +12V < 10.6 V (UV), OUTB low if +12V > 13.3 V (OV). Drives U13 ENA/ENB."
 			(at 60.96 269.24 0)
 			(hide yes)
@@
 			)
 		)
-		(property "Value" "1M"
+		(property "Value" "150k"
 			(at 41.656 262.89 0)
 			(show_name no)
@@
 			)
 		)
-		(property "Description" "TPS3700 window divider top (1 %)"
+		(property "Description" "TPS3700 window divider top (1 %): 150k"
 			(at 43.18 261.62 0)
 			(hide yes)
@@
 			)
 		)
-		(property "Value" "6.04k"
+		(property "Value" "1.2k"
 			(at 41.656 270.51 0)
 			(show_name no)
@@
 			)
 		)
-		(property "Description" "TPS3700 window divider middle (1 %): UV 11.0 V rising / 10.9 V falling"
+		(property "Description" "TPS3700 window divider middle (1 %): UV 10.6 V rising / 10.4 V falling"
 			(at 43.18 269.24 0)
 			(hide yes)
@@
 			)
 		)
-		(property "Value" "31.6k"
+		(property "Value" "4.7k"
 			(at 41.656 275.59 0)
 			(show_name no)
@@
 			)
 		)
-		(property "Description" "TPS3700 window divider bottom (1 %): OV 13.1 V rising"
+		(property "Description" "TPS3700 window divider bottom (1 %): OV 13.3 V rising"
 			(at 43.18 274.32 0)
 			(hide yes)

Commit message: Pico BNCs: Kinghelm KH-BNC50-3511 as the default part
- J7/J8/J12: Kinghelm KH-BNC50-3511 (C2837587, ~$0.93) replaces the
  Amphenol B6252HB-NPP3G-50 (C22457552, ~$3.61). 50 ohm only; never the
  KH-BNC75-3511. Saves about $34 per 5-board order.
- New footprint PiDG_Local:BNC_Kinghelm_KH-BNC50-3511_Horizontal, made
  from the board instance: Amphenol pad pattern (Kinghelm drawing matches
  within 0.04 mm), pin holes 0.89 -> 0.90 mm (Kinghelm recommended size),
  post holes 2.01 mm unchanged. 3D model is still the Amphenol body.
- Schematic and board fields (footprint, datasheet, description), BOMs,
  CPL, fp-lib-table description, Hardware.md and JLC_ORDER.md updated:
  test-fit two parts and check shell-to-GND continuity before release;
  tip ~20.6 mm past the edge, axis ~6.6 mm up (measure on first board).
- Zones refilled; gerbers, drill files and gerber zip regenerated.
  DRC/ERC: no new findings against the previous commit.

Co-Authored-By: Claude Opus 5.5 <noreply@anthropic.com>
Parts:
- J12, J7, J8: footprint Connector_Coaxial:BNC_Amphenol_B6252HB-NPP3G-50_Horizontal -> PiDG_Local:BNC_Kinghelm_KH-BNC50-3511_Horizontal
Changed lines of the file:
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@@
 			)
 		)
-		(property "Footprint" "Connector_Coaxial:BNC_Amphenol_B6252HB-NPP3G-50_Horizontal"
+		(property "Footprint" "PiDG_Local:BNC_Kinghelm_KH-BNC50-3511_Horizontal"
 			(at 358.14 124.46 0)
 			(hide yes)
@@
 			)
 		)
-		(property "Datasheet" ""
+		(property "Datasheet" "https://wmsc.lcsc.com/wmsc/upload/file/pdf/v2/lcsc/2211231430_Shenzhen-Kinghelm-Elec-KH-BNC50-3511_C2837587.pdf"
 			(at 358.14 124.46 0)
 			(hide yes)
@@
 			)
 		)
-		(property "Description" "coaxial connector (BNC, SMA, SMB, SMC, Cinch/RCA, LEMO, ...)"
+		(property "Description" "BNC 50 ohm right-angle jack, Kinghelm KH-BNC50-3511 (LCSC C2837587). Never the 75 ohm KH-BNC75-3511."
 			(at 358.14 124.46 0)
 			(hide yes)
@@
 			)
 		)
-		(property "Footprint" "Connector_Coaxial:BNC_Amphenol_B6252HB-NPP3G-50_Horizontal"
+		(property "Footprint" "PiDG_Local:BNC_Kinghelm_KH-BNC50-3511_Horizontal"
 			(at 157.48 180.34 0)
 			(hide yes)
@@
 			)
 		)
-		(property "Datasheet" ""
+		(property "Datasheet" "https://wmsc.lcsc.com/wmsc/upload/file/pdf/v2/lcsc/2211231430_Shenzhen-Kinghelm-Elec-KH-BNC50-3511_C2837587.pdf"
 			(at 157.48 180.34 0)
 			(hide yes)
@@
 			)
 		)
-		(property "Description" "coaxial connector (BNC, SMA, SMB, SMC, Cinch/RCA, LEMO, ...)"
+		(property "Description" "BNC 50 ohm right-angle jack, Kinghelm KH-BNC50-3511 (LCSC C2837587). Never the 75 ohm KH-BNC75-3511."
 			(at 157.48 180.34 0)
 			(hide yes)
@@
 			)
 		)
-		(property "Footprint" "Connector_Coaxial:BNC_Amphenol_B6252HB-NPP3G-50_Horizontal"
+		(property "Footprint" "PiDG_Local:BNC_Kinghelm_KH-BNC50-3511_Horizontal"
 			(at 213.36 180.34 0)
 			(hide yes)
@@
 			)
 		)
-		(property "Datasheet" ""
+		(property "Datasheet" "https://wmsc.lcsc.com/wmsc/upload/file/pdf/v2/lcsc/2211231430_Shenzhen-Kinghelm-Elec-KH-BNC50-3511_C2837587.pdf"
 			(at 213.36 180.34 0)
 			(hide yes)
@@
 			)
 		)
-		(property "Description" "coaxial connector (BNC, SMA, SMB, SMC, Cinch/RCA, LEMO, ...)"
+		(property "Description" "BNC 50 ohm right-angle jack, Kinghelm KH-BNC50-3511 (LCSC C2837587). Never the 75 ohm KH-BNC75-3511."
 			(at 213.36 180.34 0)
 			(hide yes)
