File: PiDG_Pico.kicad_pcb (KiCad board)
At the start: 4 copper layers, 126 x 126 mm, 84 parts, among them J1 Conn_02x05_Odd_Even, J10 Trig, J11 Laser Enable, J12 Pixel Reset, J14 Pico Socket A, J15 Pico Socket B, J16 Laser En/PWM Trig/GND, J17 USB-C PD in, J18 Laser 1 mode, J19 Laser 2 mode, J2 Conn_02x05_Odd_Even, J3 Conn_02x05_Odd_Even, J4 Conn_02x05_Odd_Even, J5 Conn_02x05_Odd_Even, J6 Conn_02x05_Odd_Even, J7 Laser 1, J8 Laser 2, U1 74LVC1G04, U10 74AHCT1G08, U12 74LVC1G17, U13 UCC27524, U14 CH224A, U15 AP63205WU, U16 LM66100, U17 LT3065EDD, U18 TPS3700DDC, U2 SN74LVC04AD, U3 74LVC1G00, U4 SN74LVC04AD, U5 74LVC1G04, U6 SN74LVC04AD, U7 74AHCT1G08, U8 74AHCT1G08, U9 NCP718xSN180

Commit message: SYNC: 1 MHz from the RP2350 clock generator on GP15 (was PIO on GP10)
Firmware
- New sync_clock.h/.cpp: clk_gpout1 divides clk_sys straight onto GP15
  (16.16 divider, exactly 150 at 150 MHz, DC50 duty correction): an exact,
  jitter-free 1 MHz square wave. The pin is held LOW until it starts.
- Only GP13/15/21 (GP23-25 internal on the Pico 2 W) have a clk_gpout
  function; GP13 is CH1, so SYNC moves to GP15. GPIO9 has none.
- Remove the PIO toggle program and SyncChannel; pio1 is no longer used.
- pulse_timing.h: syncDiv is the 16.16 clock-generator divider; STATUS
  prints "divider 150+0/65536". GUI parser accepts any I+F/N divider.
- Timing checks: harness/check_sync.py updated; all six checks pass.

Hardware
- Schematic: PWM_1MHz on J14/U11 pin 20 (GP15); pin 14 (GP10) no-connect.
- Board: PWM_1MHz leaves J14 pad 20 on F.Cu (B.Cu there runs between the
  CH2/CH1 traces) and drops through a via to the existing B.Cu trunk at
  x = 155 mm; old pad-14 stub removed. No other signal within 2 mm of the
  new section; PIXRST_GATE 17 mm away; solid In1/In2 planes between the
  trunk and R17/R18. Zones refilled; gerbers, drill files and zip
  regenerated; JLC BOM/CPL unchanged.
- Docs: README, Hardware.md (pin tables, signal chain, timing), board.h.

Checks: ERC 0; DRC 0 errors, 0 unconnected; pico2w and pico2 build with
0 warnings; Markdown links resolve.

Co-Authored-By: Claude Opus 5.5 <noreply@anthropic.com>
Connections:
- J14 pad 14: PWM_1MHz -> (no net)
- J14 pad 20: (no net) -> PWM_1MHz
Routing:
- net PWM_1MHz: vias 1 -> 2
Changed lines of the file:
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@@
 			(layers "*.Cu" "*.Mask")
 			(remove_unused_layers no)
-			(net "PWM_1MHz")
 		)
 		(pad "15" thru_hole circle
@@
 			(layers "*.Cu" "*.Mask")
 			(remove_unused_layers no)
+			(net "PWM_1MHz")
 		)
 		(embedded_fonts no)
@@
 		(net "PWM_1MHz")
 	)
+	(segment
+		(start 160.01 80.64)
+		(end 155 80.64)
+		(width 0.5)
+		(layer "F.Cu")
+		(net "PWM_1MHz")
+	)
+	(via
+		(at 155 80.64)
+		(size 0.6)
+		(drill 0.3)
+		(layers "F.Cu" "B.Cu")
+		(net "PWM_1MHz")
+	)
 	(via
 		(at 155 110.53)
@@
 	)
 	(segment
-		(start 160.015 65.405)
-		(end 155 65.405)
+		(start 155 80.64)
+		(end 155 110.53)
 		(width 0.5)
 		(layer "B.Cu")
@@
 	(segment
 		(start 155 65.405)
-		(end 155 110.53)
+		(end 155 80.64)
 		(width 0.5)
 		(layer "B.Cu")

Commit message: Board: clock jumper J20 with R29 series resistor; Rev 1; schematic tidy
- J20 (2-pin header, C32713268) left of J14: pin 1 CLK_SEL_JMP -> R29 1k
  (C17513) -> CLK_SEL = GP10 (J14 pad 14), pin 2 GND. Shunt fitted =
  300 MHz, open = 150 MHz. R29 limits the current to about 3.3 mA if GP10
  is driven with the shunt fitted (firmware before 5dfedd5 drove GP10 as
  SYNC); a fitted shunt still reads about 0.1 V. No capacitor on CLK_SEL.
- PCB: J20 at (152.4, 65.405), R29 inline on F.Cu, silkscreen CLOCK JUMPER /
  OPEN = 150 MHz / FIT = 300 MHz (OVERCLOCK). Zones refilled. DRC: 0
  violations, 0 unconnected; schematic parity: no real net mismatches.
- Rev 1 (no board built yet): schematic title block rev 03 -> 1, dated
  2026-10-20; PCB title block added, so the gerbers carry revision 1.
- Schematic tidy pass, netlist unchanged apart from R29: field, label and
  power-symbol overlaps fixed; R6/R7 moved clear of the sheet frame; C9/C10
  drawn with +12V on top; duplicate labels removed; U11 pin 18 GND as a
  global label like the other GND pins. ERC: 0.
- Fab: gerbers, drill files and zip regenerated; master BOM, JLC BOM
  (43 lines) and CPL (82 parts, via tools/jlc_cpl) updated; 5 loose shunts.
- Docs: Hardware.md, README.md, JLC_ORDER.md, board.h and clock_mode.cpp
  comments; notes/kicad-clock-jumper.md removed (all items done).
  Hardware.md now states 82 placed parts and 0.5 mm copper-to-edge (the
  board rule).

Co-Authored-By: Claude Opus 5.5 <noreply@anthropic.com>
Parts:
- added J20: Clock jumper, Connector_PinHeader_2.54mm:PinHeader_1x02_P2.54mm_Vertical, F.Cu at (152.4, 65.4)
- added R29: 1k, Resistor_SMD:R_0805_2012Metric_Pad1.20x1.40mm_HandSolder, F.Cu at (156.2, 65.4)
Connections:
- J14 pad 14: (no net) -> CLK_SEL
Routing:
- net CLK_SEL_JMP: track 0.00 -> 2.81 mm
- net CLK_SEL: track 0.00 -> 2.80 mm
Other:
- board text added: "(OVERCLOCK)"
- board text added: "CLOCK JUMPER"
- board text added: "FIT = 300 MHz"
- board text added: "OPEN = 150 MHz"

Commit message: Board: J12 becomes External Sync Out; remove J16 and the external pixel-reset input
- J12 BNC now outputs a copy of the camera trigger (PWM_TRIG_TAP) through a
  third UCC27524 channel (U19), built like Laser 1: R30 68 ohm 2 W, J21 mode
  jumper with R31 47 ohm / R32 82 ohm (50 ohm or Hi-Z), gated by LASER_PWR_OK.
- J16 (laser-enable / trigger monitor header) removed with its traces;
  PWM_TRIG_TAP shortened from ~122 mm to ~59 mm.
- External pixel-reset input removed (U12, R5, C8); U3 inputs tied to
  PIXRST_GATE, so pixel reset comes only from the Pico (GP16).
- Fab outputs, BOM, JLC BOM/CPL (85 parts, 41 lines) and order notes updated;
  firmware/GUI strings no longer mention J12 as an input.

ERC 0, DRC 0/0. Revision stays 1.

Co-Authored-By: Claude Opus 5.5 (1M context) <noreply@anthropic.com>
Parts:
- removed C8: 0.1uF, Capacitor_SMD:C_0805_2012Metric_Pad1.18x1.45mm_HandSolder
- removed J16: Laser En/PWM Trig/GND, PiDG_Local:PinHeader_1x03_P2.54mm_Horizontal_EdgeTrim
- removed R5: 3k3, Resistor_SMD:R_0805_2012Metric_Pad1.20x1.40mm_HandSolder
- removed U12: 74LVC1G17, Package_TO_SOT_SMD:SOT-23-5_HandSoldering
- added C21: 0.1uF, Capacitor_SMD:C_0805_2012Metric_Pad1.18x1.45mm_HandSolder, F.Cu at (216.6, 128.6)
- added C22: 10uF 50V, Capacitor_SMD:C_1206_3216Metric_Pad1.33x1.80mm_HandSolder, F.Cu at (215.9, 121.6)
- added J21: Ext sync mode, Connector_PinHeader_2.54mm:PinHeader_1x03_P2.54mm_Vertical, F.Cu at (236.5, 118.1)
- added R30: 68, Resistor_SMD:R_2512_6332Metric_Pad1.40x3.35mm_HandSolder, F.Cu at (223.9, 126.9)
- added R31: 47, Resistor_SMD:R_2512_6332Metric_Pad1.40x3.35mm_HandSolder, F.Cu at (230.1, 120.7)
- added R32: 82, Resistor_SMD:R_2512_6332Metric_Pad1.40x3.35mm_HandSolder, F.Cu at (233.4, 127.2)
- added U19: UCC27524, Package_SO:SOIC-8_3.9x4.9mm_P1.27mm, F.Cu at (210.9, 128.0)
- J12: value Pixel Reset -> Ext Sync Out
Connections:
- J12 pad 1: PIXRST_IN -> EXT_SYNC_OUT
- U3 pad 2: PIXRST -> PIXRST_GATE
Routing:
- net +3V3: track 142.9 -> 56.9 mm, vias 2 -> 0
- net PWM_TRIG_TAP: track 122.2 -> 58.5 mm
- net PIXRST: track 61.7 -> 0.00 mm, vias 2 -> 0
- net +12V: track 64.0 -> 121.6 mm, vias 2 -> 4
- net LASER_PWR_OK: track 26.2 -> 79.2 mm, vias 0 -> 2
- net LASER_EN_TAP: track 44.2 -> 5.65 mm
- net EXT_SYNC_DRIVE: track 0.00 -> 19.7 mm
- net PIXRST_IN: track 12.6 -> 0.00 mm
- net EXT_SYNC_OUT: track 0.00 -> 11.9 mm
- net EXT_SYNC_DRIVE_RAW: track 0.00 -> 7.53 mm
- net GND: track 70.1 -> 76.0 mm, vias 83 -> 85
- net EXT_SYNC_TERM: track 0.00 -> 4.02 mm
- net PIXRST_GATE: track 31.3 -> 32.3 mm
Other:
- board text added: "EXT SYNC OUT"
- board text removed: "EN"
- board text removed: "EN IN: PULL LOW = LASERS OFF"
- board text removed: "J16: NEVER FIT A SHUNT"
- board text removed: "NOT FAIL-SAFE: E-STOP ON J11"
- board text removed: "PIXEL RESET"
- board text removed: "TRIG"
- board text removed: "TRIG OUT: CAMERA TRIGGER (MONITOR)"
