File: PiDG_Pico.kicad_sch (KiCad schematic)
At the start: 81 parts, among them J1 Conn_02x05_Odd_Even, J10 Trig, J11 Laser Enable, J12 Pixel Reset, J14 Pico Socket A, J15 Pico Socket B, J16 Laser En/PWM Trig/GND, J17 USB-C PD in, J18 Laser 1 mode, J19 Laser 2 mode, J2 Conn_02x05_Odd_Even, J3 Conn_02x05_Odd_Even, J4 Conn_02x05_Odd_Even, J5 Conn_02x05_Odd_Even, J6 Conn_02x05_Odd_Even, J7 Laser 1, J8 Laser 2, U1 74LVC1G04, U10 74AHCT1G08, U11 Raspberry Pi Pico 2 W, U12 74LVC1G17, U13 UCC27524, U14 CH224A, U15 AP63205WU, U16 LM66100, U17 LT3065EDD, U18 TPS3700DDC, U2 SN74LVC04AD, U3 74LVC1G00, U4 SN74LVC04AD, U5 74LVC1G04, U6 SN74LVC04AD, U7 74AHCT1G08, U8 74AHCT1G08, U9 NCP718xSN180

Commit message: Clean up: remove Teensy leftovers, redundant files and stale references
- Teensy: remove libs/teensy.* and their lib-table entries, the orphaned
  cached teensy:Teensy4.1 symbol in the schematic, and all Teensy mentions
  in Hardware.md, README, src comments and part descriptions.
- Redundant files: delete the KiCad-format PiDG_Pico_CPL.csv (the JLC CPL
  in fab/jlc/ is the only placement file), stale erc.json and
  PiDG_Pico_drc_violations.json, libs/RPi_Pico.pretty (only used by the
  unplaced U11's footprint field, now cleared), and the empty PlatformIO
  template folders include/, lib/, test/.
- Move the master BOM to fab/PiDG_Pico_BOM.csv; docs updated.
- fp-lib-table: drop 10 standard-library entries with an absolute
  "C:/Program Files/KiCad" path (the global table provides them); ERC
  library warnings 68 -> 0.
- Remove the other machine's MCP config (.mcp.json, .vscode/mcp.json).
- Ignore *.kicad_prl (per-user KiCad view settings) and KiCad check
  reports; stale doc references (HARDWARE_DESIGN.md) fixed.
- Checks: netlist connectivity identical; ERC 0; DRC 0 errors (parity
  notes only); all Markdown links resolve; pio run -e pico2w succeeds.

Co-Authored-By: Claude Opus 5.5 <noreply@anthropic.com>
Parts:
- U11: footprint RPi_Pico:RPi_Pico2W_SMD_TH -> (none)
Changed lines of the file:
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@@
 			)
 		)
-		(property "Footprint" "RPi_Pico:RPi_Pico2W_SMD_TH"
+		(property "Footprint" ""
 			(at 137.16 251.46 0)
 			(hide yes)
@@
 			)
 		)
-		(property "Description" "RP2350 + CYW43439 (wireless unused) module -- replaces the Teensy 4.1 (see HARDWARE_DESIGN.md)"
+		(property "Description" "RP2350 + CYW43439 (wireless unused) module, socketed in J14/J15 (see Hardware.md)"
 			(at 137.16 251.46 0)
 			(hide yes)
@@
 			)
 		)
-		(property "Description" "Dual 50-ohm-matched laser trigger driver (see HARDWARE_DESIGN.md 2.2)"
+		(property "Description" "Dual laser trigger driver, UCC27524 (see Hardware.md, Laser outputs)"
 			(at 378.46 43.18 0)
 			(hide yes)

Commit message: SYNC: 1 MHz from the RP2350 clock generator on GP15 (was PIO on GP10)
Firmware
- New sync_clock.h/.cpp: clk_gpout1 divides clk_sys straight onto GP15
  (16.16 divider, exactly 150 at 150 MHz, DC50 duty correction): an exact,
  jitter-free 1 MHz square wave. The pin is held LOW until it starts.
- Only GP13/15/21 (GP23-25 internal on the Pico 2 W) have a clk_gpout
  function; GP13 is CH1, so SYNC moves to GP15. GPIO9 has none.
- Remove the PIO toggle program and SyncChannel; pio1 is no longer used.
- pulse_timing.h: syncDiv is the 16.16 clock-generator divider; STATUS
  prints "divider 150+0/65536". GUI parser accepts any I+F/N divider.
- Timing checks: harness/check_sync.py updated; all six checks pass.

Hardware
- Schematic: PWM_1MHz on J14/U11 pin 20 (GP15); pin 14 (GP10) no-connect.
- Board: PWM_1MHz leaves J14 pad 20 on F.Cu (B.Cu there runs between the
  CH2/CH1 traces) and drops through a via to the existing B.Cu trunk at
  x = 155 mm; old pad-14 stub removed. No other signal within 2 mm of the
  new section; PIXRST_GATE 17 mm away; solid In1/In2 planes between the
  trunk and R17/R18. Zones refilled; gerbers, drill files and zip
  regenerated; JLC BOM/CPL unchanged.
- Docs: README, Hardware.md (pin tables, signal chain, timing), board.h.

Checks: ERC 0; DRC 0 errors, 0 unconnected; pico2w and pico2 build with
0 warnings; Markdown links resolve.

Co-Authored-By: Claude Opus 5.5 <noreply@anthropic.com>
Connections:
- net PWM_1MHz: now also J14.20 (Pin_20), U11.20 (GP15); no longer J14.14 (Pin_14), U11.14 (GP10)
Changed lines of the file:
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@@
 	)
 	(no_connect
-		(at 194.31 275.59)
+		(at 194.31 260.35)
 	)
 	(no_connect
@@
 	)
 	(no_connect
-		(at 116.84 275.59)
+		(at 116.84 260.35)
 	)
 	(no_connect
@@
 	(wire
 		(pts
-			(xy 116.84 260.35) (xy 114.3 260.35)
+			(xy 116.84 275.59) (xy 114.3 275.59)
 		)
 		(stroke
@@
 	)
 	(label "PWM_1MHz"
-		(at 194.31 260.35 180)
+		(at 194.31 275.59 180)
 		(effects
 			(font
@@
 	)
 	(label "PWM_1MHz"
-		(at 114.3 260.35 0)
+		(at 114.3 275.59 0)
 		(effects
 			(font

Commit message: Board: clock jumper J20 with R29 series resistor; Rev 1; schematic tidy
- J20 (2-pin header, C32713268) left of J14: pin 1 CLK_SEL_JMP -> R29 1k
  (C17513) -> CLK_SEL = GP10 (J14 pad 14), pin 2 GND. Shunt fitted =
  300 MHz, open = 150 MHz. R29 limits the current to about 3.3 mA if GP10
  is driven with the shunt fitted (firmware before 5dfedd5 drove GP10 as
  SYNC); a fitted shunt still reads about 0.1 V. No capacitor on CLK_SEL.
- PCB: J20 at (152.4, 65.405), R29 inline on F.Cu, silkscreen CLOCK JUMPER /
  OPEN = 150 MHz / FIT = 300 MHz (OVERCLOCK). Zones refilled. DRC: 0
  violations, 0 unconnected; schematic parity: no real net mismatches.
- Rev 1 (no board built yet): schematic title block rev 03 -> 1, dated
  2026-10-20; PCB title block added, so the gerbers carry revision 1.
- Schematic tidy pass, netlist unchanged apart from R29: field, label and
  power-symbol overlaps fixed; R6/R7 moved clear of the sheet frame; C9/C10
  drawn with +12V on top; duplicate labels removed; U11 pin 18 GND as a
  global label like the other GND pins. ERC: 0.
- Fab: gerbers, drill files and zip regenerated; master BOM, JLC BOM
  (43 lines) and CPL (82 parts, via tools/jlc_cpl) updated; 5 loose shunts.
- Docs: Hardware.md, README.md, JLC_ORDER.md, board.h and clock_mode.cpp
  comments; notes/kicad-clock-jumper.md removed (all items done).
  Hardware.md now states 82 placed parts and 0.5 mm copper-to-edge (the
  board rule).

Co-Authored-By: Claude Opus 5.5 <noreply@anthropic.com>
Parts:
- added J20: Clock jumper, Connector_PinHeader_2.54mm:PinHeader_1x02_P2.54mm_Vertical, symbol Connector:Conn_01x02_Pin
- added R29: 1k, Resistor_SMD:R_0805_2012Metric_Pad1.20x1.40mm_HandSolder, symbol Device:R_Small
Connections:
- net GND: now also J20.2 (Pin_2)
- net CLK_SEL: now reaches U11.14 (GP10)
- net CLK_SEL: now also J14.14 (Pin_14), R29.2
- new net CLK_SEL_JMP: J20.1 (Pin_1), R29.1
- no-connect marks 93 -> 91
Other:
- note added: "J20 clock jumper on GP10, read at every start. Shunt fitted: 300 MHz. Open: 150 MHz (rated). R29: protects GP10 if driven into the shunt. Internal pull-up only: no capacitor on CLK_SEL."
- moved on the sheet: C10, C9, R19, R6, R7

Commit message: Board: J12 becomes External Sync Out; remove J16 and the external pixel-reset input
- J12 BNC now outputs a copy of the camera trigger (PWM_TRIG_TAP) through a
  third UCC27524 channel (U19), built like Laser 1: R30 68 ohm 2 W, J21 mode
  jumper with R31 47 ohm / R32 82 ohm (50 ohm or Hi-Z), gated by LASER_PWR_OK.
- J16 (laser-enable / trigger monitor header) removed with its traces;
  PWM_TRIG_TAP shortened from ~122 mm to ~59 mm.
- External pixel-reset input removed (U12, R5, C8); U3 inputs tied to
  PIXRST_GATE, so pixel reset comes only from the Pico (GP16).
- Fab outputs, BOM, JLC BOM/CPL (85 parts, 41 lines) and order notes updated;
  firmware/GUI strings no longer mention J12 as an input.

ERC 0, DRC 0/0. Revision stays 1.

Co-Authored-By: Claude Opus 5.5 (1M context) <noreply@anthropic.com>
Parts:
- removed C8: 0.1uF, Capacitor_SMD:C_0805_2012Metric_Pad1.18x1.45mm_HandSolder, symbol Device:C
- removed J16: Laser En/PWM Trig/GND, PiDG_Local:PinHeader_1x03_P2.54mm_Horizontal_EdgeTrim, symbol Connector:Conn_01x03_Pin
- removed R5: 3k3, Resistor_SMD:R_0805_2012Metric_Pad1.20x1.40mm_HandSolder, symbol Device:R_Small
- removed U12: 74LVC1G17, Package_TO_SOT_SMD:SOT-23-5_HandSoldering, symbol 74xGxx:74LVC1G17
- added C21: 0.1uF, Capacitor_SMD:C_0805_2012Metric_Pad1.18x1.45mm_HandSolder, symbol Device:C
- added C22: 10uF 50V, Capacitor_SMD:C_1206_3216Metric_Pad1.33x1.80mm_HandSolder, symbol Device:C
- added J21: Ext sync mode, Connector_PinHeader_2.54mm:PinHeader_1x03_P2.54mm_Vertical, symbol Connector:Conn_01x03_Pin
- added R30: 68, Resistor_SMD:R_2512_6332Metric_Pad1.40x3.35mm_HandSolder, symbol Device:R_Small
- added R31: 47, Resistor_SMD:R_2512_6332Metric_Pad1.40x3.35mm_HandSolder, symbol Device:R_Small
- added R32: 82, Resistor_SMD:R_2512_6332Metric_Pad1.40x3.35mm_HandSolder, symbol Device:R_Small
- added U19: UCC27524, Package_SO:SOIC-8_3.9x4.9mm_P1.27mm, symbol PiDG_Local:UCC27524
- J12: value Pixel Reset -> Ext Sync Out
Connections:
- net PIXRST is gone; now on net PIXRST_GATE: U3.2
- net +12V: now also C21.2, C22.2, U19.6 (VDD)
- net GND: now also C21.1, C22.1, R32.2, U19.3 (GND), U19.4 (INB)
- net LASER_PWR_OK: now also U19.1 (ENA), U19.8 (ENB)
- net PWM_TRIG_TAP: now also U19.2 (INA)
- net PIXRST_IN renamed EXT_SYNC_OUT
- net EXT_SYNC_OUT: now also J21.2 (Pin_2), R31.2
- new net EXT_SYNC_DRIVE: J21.1 (Pin_1), R30.2, R31.1
- new net EXT_SYNC_DRIVE_RAW: R30.1, U19.7 (OUTA)
- new net EXT_SYNC_TERM: J21.3 (Pin_3), R32.1
- no-connect marks 91 -> 92
Other:
- note added: "EXT SYNC OUTPUT (J12)"
- note added: "Output mode, one shunt per channel (J18 = Laser 1, J19 = Laser 2, J21 = Ext sync): 1-2 50 ohm: series 47R bypassed. 4.54-5.14 V into a 50 ohm load (PicoLas LDP-V); ~12 V open circuit. 2-3 Hi-Z: 68R + 47R in series, 82R shunt -> 4.55-5.08 V open circuit from a 47-50 ohm source (back-terminated, no overshoot on long cables); 2.3-2.6 V into 50 ohm: an LDP-V will not trigger. No shunt: ~12 V open cir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"
- note added: "U3 = NAND with both inputs on PIXRST_GATE: via U4 the cameras get TDRSTN = PIXRST_GATE. Only the Pico (GP16, PIXGATE) resets the pixels. R24 holds the gate high otherwise."
- note removed: "Output mode, one shunt per channel (J18 = Laser 1, J19 = Laser 2): 1-2 50 ohm: series 47R bypassed. 4.54-5.14 V into a 50 ohm load (PicoLas LDP-V); ~12 V open circuit. 2-3 Hi-Z: 68R + 47R in series, 82R shunt -> 4.55-5.08 V open circuit from a 47-50 ohm source (back-terminated, no overshoot on long cables); 2.3-2.6 V into 50 ohm: an LDP-V will not trigger. No shunt: ~12 V open circuit, ~3.5 V int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"
- note removed: "U3 = NAND. Via U4 the cameras get TDRSTN = PIXRST AND PIXRST_GATE: J12 or the Pico (GP16, PIXGATE) resets the pixels. R24 holds the gate high otherwise."
- moved on the sheet: J12
